Commit message: 清除mid360驱动，增加e1r雷达配置文件，修改tf等适配新激光雷达和imu,启动方式集成到xj_robot_bringup包中的robot.launch.py，启动前需要启动雷达驱动

File: src/nav/xjrobot_base/urdf/sensors/lidar_3d.urdf.xacro (robot description, xacro)
@@ -15,5 +15,5 @@
            实机版本当前与仿真保持一致，xyz=(0.285, 0, 0.165), rpy=(0, 0, 0)。
            后续调整 3D 雷达安装位置，请修改这里。 -->
-      <origin xyz="0.24 0 0.02" rpy="0.0 0.0 0.0" />
+      <origin xyz="0.17262 0 0.0" rpy="0.0 0.0 0.0" />
       <parent link="base_link" />
       <child link="lidar_3d_link" />
